File: keyboard_featherwing.kicad_pcb (KiCad board)
At the start: 2 copper layers, 68 x 100 mm, 58 parts, among them J3 Micro_SD_Card_Det, J7 Conn_Stemma_QT, Q1 BSS138, Q2 BSS138, SW1 SW_EN, SW2 SW_RIGHT1, SW3 SW_LEFT1, SW4 SW_RIGHT2, SW5 SW_LEFT2, U1 5-Way_Switch, U2 BBQ10KBD, U4 ER-TFT02X, U5 STMPE811, U6 Adafruit_Feather_2X, U7 ATSAMD20G16A, U8 74AHCT1G125

Commit message: Production HW Rev 2
Parts:
- removed the G*** at (152.4, 124.4)
- removed U5: STMPE811, Package_DFN_QFN:QFN-16-1EP_3x3mm_P0.5mm_EP1.75x1.75mm
- added ?: , buzzardLabel, F.Cu at (110.2, 102.7)
- added ?: , buzzardLabel, F.Cu at (166.4, 115.1)
- added ?: , buzzardLabel, F.Cu at (150.1, 70.7)
- added ?: , buzzardLabel, F.Cu at (150.3, 78.2)
- added ?: , buzzardLabel, F.Cu at (160.0, 110.9)
- added ?: , buzzardLabel, F.Cu at (153.4, 115.1)
- added ?: , buzzardLabel, F.Cu at (149.4, 65.7)
- added ?: , buzzardLabel, F.Cu at (127.3, 92.2)
- added ?: , buzzardLabel, F.Cu at (136.9, 137.6)
- added ?: , buzzardLabel, F.Cu at (125.4, 47.6)
- added ?: , buzzardLabel, F.Cu at (156.1, 73.2)
- added ?: , buzzardLabel, F.Cu at (156.5, 68.2)
- added ?: , buzzardLabel, F.Cu at (118.4, 55.5)
- added ?: , buzzardLabel, F.Cu at (150.0, 68.2)
- added ?: , buzzardLabel, F.Cu at (156.1, 75.7)
- added ?: , buzzardLabel, F.Cu at (157.6, 115.1)
- added ?: , buzzardLabel, F.Cu at (145.4, 115.1)
- added ?: , buzzardLabel, F.Cu at (149.9, 73.2)
- added ?: , buzzardLabel, F.Cu at (118.5, 53.9)
- added ?: , buzzardLabel, F.Cu at (135.7, 47.6)
- added ?: , buzzardLabel, F.Cu at (162.7, 49.9)
- added ?: , buzzardLabel, F.Cu at (156.8, 78.2)
- added ?: , buzzardLabel, F.Cu at (110.2, 104.2)
- added ?: , buzzardLabel, F.Cu at (145.9, 56.0)
- added ?: , buzzardLabel, F.Cu at (162.3, 115.1)
- added ?: , buzzardLabel, F.Cu at (150.0, 75.7)
- added ?: , buzzardLabel, F.Cu at (154.3, 86.9)
- added ?: , buzzardLabel, F.Cu at (156.4, 65.7)
- added ?: , buzzardLabel, F.Cu at (154.6, 63.3)
- added ?: , buzzardLabel, F.Cu at (156.1, 70.7)
- added ?: , buzzardLabel, F.Cu at (153.9, 63.3)
- added JP7: SB_ALS, Jumper:SolderJumper-2_P1.3mm_Bridged_RoundedPad1.0x1.5mm, F.Cu at (154.3, 63.3)
- added Q3: PT26-21C, OptoDevice_Extra:Everlight_PT26-21C, F.Cu at (160.9, 49.9)
- added R10: 10K, Resistor_SMD:R_0603_1608Metric, F.Cu at (160.8, 54.6)
- added TP11: TP_GPIO3, TestPoint:TestPoint_Pad_D2.0mm, F.Cu at (160.0, 131.4)
- added TP12: TP_GPIO4, TestPoint:TestPoint_Pad_D2.0mm, F.Cu at (160.0, 134.6)
- added TP13: TP_GPIO5, TestPoint:TestPoint_Pad_D2.0mm, F.Cu at (160.0, 137.8)
- added TP14: TP_GPIO6, TestPoint:TestPoint_Pad_D2.0mm, F.Cu at (160.0, 141.0)
- added TP8: TP_GPIO2, TestPoint:TestPoint_Pad_D2.0mm, F.Cu at (160.0, 128.3)
- added U3: TSC2004IR, Package_DFN_QFN:QFN-20-1EP_4x4mm_P0.5mm_EP2.7x2.7mm, F.Cu at (128.5, 95.5)
- JP5: value SB_STM_CS -> SB_KBD_INT
- SW1: value SW_EN -> SK-3245S-Lx-B; footprint Button_Switch_SMD:SW_SPDT_PCM12 -> Button_Switch_SMD_Extra:K3-x245S
- TP1, TP10, TP2, TP3, TP4, TP9: footprint TestPoint:TestPoint_Pad_D3.0mm -> TestPoint:TestPoint_Pad_D2.0mm
- TP5: value TP_STM_INT -> TP_NEOPIXEL_OUT; footprint TestPoint:TestPoint_Pad_D3.0mm -> TestPoint:TestPoint_Pad_D2.0mm
- moved TP5 52.0 mm to (118.4, 57.5)
- moved R9 45.5 mm to (162.4, 59.5), turned to 180 degrees
- moved JP3 39.7 mm to (154.3, 68.2)
- moved JP6 35.5 mm to (154.3, 65.7)
- moved JP2 35.4 mm to (154.3, 70.7)
- moved JP5 31.3 mm to (154.3, 73.2)
- moved R1 30.9 mm to (112.9, 97.8)
- moved R2 28.0 mm to (114.4, 97.8)
- moved R8 27.6 mm to (152.2, 81.2), turned to -90 degrees
- moved JP1 21.9 mm to (154.3, 75.7)
- moved TP4 20.7 mm to (145.4, 113.1)
- moved C6 11.9 mm to (123.2, 95.0), turned to 90 degrees
- moved R6 4.93 mm to (120.3, 60.6)
- moved R7 4.93 mm to (125.4, 60.6)
- moved Q2 4.93 mm to (122.9, 60.6)
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Connections:
- net /CARD_MISO renamed /CARD_CIPO
- net /CARD_MOSI renamed /CARD_COPI
- D2 pad 1: +5V -> Net-(D2-Pad1)
- D3 pad 1: +5V -> Net-(D2-Pad1)
- J3 pad 1: Net-(J3-Pad1) -> unconnected-(J3-Pad1)
- J3 pad 8: Net-(J3-Pad8) -> unconnected-(J3-Pad8)
- JP5 pad 2: /STM_CS -> /KBD_INT
- R9 pad 1: /STM_CS -> /CARD_DET
- SW1 pad 1: Net-(SW1-Pad1) -> GND
- SW1 pad 3: GND -> unconnected-(SW1-Pad3)
- TP5 pad 1: Net-(TP5-Pad1) -> Net-(D1-Pad2)
- U4 pad 39: Net-(U4-Pad39) -> unconnected-(U4-Pad39)
- U6 pad 16: Net-(U6-Pad16) -> unconnected-(U6-Pad16)
- U7 pad 15: Net-(U7-Pad15) -> /CARD_DET
- U7 pad 16: Net-(U7-Pad16) -> unconnected-(U7-Pad16)
- U7 pad 33: Net-(U7-Pad33) -> /TP_INT
- U7 pad 34: Net-(U7-Pad34) -> /LCD_BL_CTRL
- U7 pad 7: Net-(U7-Pad7) -> unconnected-(U7-Pad7)
Routing:
- net GND: track 90.1 -> 47.4 mm, vias 144 -> 100
- net Net-(TP14-Pad1): track 0.00 -> 41.8 mm
- net /GPIO11: track 60.6 -> 19.2 mm, vias 2 -> 0
- net /NEOPIXEL: track 5.28 -> 45.9 mm, vias 0 -> 2
- net Net-(TP13-Pad1): track 0.00 -> 39.9 mm
- net /TP_INT: track 0.00 -> 37.3 mm, vias 0 -> 2
- net /LCD_BL_CTRL: track 42.4 -> 79.6 mm, vias 2 -> 4
- net /GPIO10: track 54.2 -> 19.3 mm, vias 2 -> 0
- net Net-(TP12-Pad1): track 0.00 -> 34.7 mm, vias 0 -> 2
- net /CARD_CIPO: track 93.7 -> 61.6 mm, vias 3 -> 2
- net Net-(TP11-Pad1): track 0.00 -> 32.1 mm, vias 0 -> 2
- net +3V3: track 280.6 -> 310.7 mm, vias 20 -> 11
- net Net-(TP8-Pad1): track 0.00 -> 29.2 mm, vias 0 -> 2
- net /CARD_CLK: track 77.2 -> 48.1 mm, vias 2 -> 0
- net /GPIO5: track 43.3 -> 18.1 mm
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Other:
- board text added: "0x1F - Keyboard"
- board text added: "0x4B - Touch IC"
- board text added: "CI"
- board text added: "CO"
- board text added: "D10: LCD DC"
- board text added: "D11: NEOPIXEL"
- board text added: "D5: Card CS"
- board text added: "D6: KBD INT"
- board text added: "D9: LCD CS"
- board text added: "Expander GPIOs:"
- board text added: "Feather GPIOs:"
- board text added: "GPIO0: Touch INT"
- board text added: "GPIO1: Card Detect"
- board text added: "GPIO2:"
- board text added: "GPIO3:"
- board text added: "GPIO4:"
- board text added: "GPIO5:"
- board text added: "GPIO6:"
- board text added: "I_{2}C:"
- board text added: "JLCJLCJLCJLC"
- board text added: "Keyboard FeatherWing by arturo182 Feb 2021"
- board text removed: "3.3V"
- board text removed: "CARD CS"
- board text removed: "CLK"
- board text removed: "GPIOs: D5: CARD CS D6: STMP CS D9: LCD CS D10: LCD DC D11: NEOPIXEL I2C: 0x1F - Keyboard"
- board text removed: "IO"
- board text removed: "KBD IC SWD"
- board text removed: "KBD TX"
- board text removed: "Keyboard FeatherWing by arturo182 April 2020"
- board text removed: "LCD CS"
- board text removed: "LCD DC"
- board text removed: "MI"
- board text removed: "MIC"
- board text removed: "MIC EN"
- board text removed: "MO"
- board text removed: "NEOPIXEL"
- board text removed: "OFF"
- board text removed: "ON"
- board text removed: "Qwiic STEMMA QT"
- board text removed: "STMP CS"
- board text removed: "STMP INT"
